File: ECC83-daughterboard/HVBoost.kicad_sch (KiCad schematic)
At the start: 17 parts, among them Q1 IRF7495, T2 EP7_750310020, U3 LT3757AEDD

Commit message: added some design notes for future self
Other:
- note added: "Recommended BOM, version I would actually build first U1 LT3757AEDD#PBF or LT3757AEMSE#PBF Use the DFN if you want the smallest PCB. LT3757A is a boost/flyback/SEPIC/inverting controller, operates from 2.9 V to 40 V, drives an external low-side NMOS from its internal 7.2 V supply, and is intended for exactly this kind of topology. T1 Coilcraft DA2032-ALD This is the off-the-shelf transformer I wo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"
- note added: "https://www.analog.com/media/en/technical-documentation/data-sheets/lt3757-3757a.pdf"

Commit message: HV boost schematic in line with datasheet, half-calculated values
Parts:
- removed D3: MUR160, Diode_THT:D_DO-41_SOD81_P10.16mm_Horizontal, symbol Diode:1N4001
- removed Q1: IRF7495, Package_SO:SOIC-8_3.9x4.9mm_P1.27mm, symbol Transistor_FET:IRF7403
- removed T2: EP7_750310020, WE-PoE:T_Wurth_WE-PoE-EP7, symbol WE-PoE:EP7_750310020
- added C1, C2: 10u, Capacitor_SMD:C_0603_1608Metric_Pad1.08x0.95mm_HandSolder, symbol Device:C
- added C7: 47u 25V, Capacitor_SMD:C_0603_1608Metric_Pad1.08x0.95mm_HandSolder, symbol Device:C
- added C8: C, Capacitor_SMD:C_0603_1608Metric_Pad1.08x0.95mm_HandSolder, symbol Device:C
- added D1: ES1G-13-F, Diode_SMD:D_SMA_Handsoldering, symbol Device:D_Schottky
- added Q1: BSC340N08NS3G, Package_TO_SOT_SMD:TDSON-8-1, symbol Transistor_FET:BSC340N08NS3G
- added R9: 20k 1%, Resistor_SMD:R_0603_1608Metric, symbol Device:R
- added U2: DA2032-AL, DA2032-AL:DA2032-AL, symbol Coilcraft:DA2032-AL
- C3: value C -> 100u
- C4: renamed from C1; value C -> 100n
- C5: value C -> 100p
- C6: value C -> 3.3n
- C9: renamed from C4; value C -> 1u 250V
- R1: value R -> 105k
- R2: value R -> 46.4
- R3: value R -> 41.2k
- R4: value R -> 18k
- R5: value R -> 0.02; footprint Resistor_SMD:R_0402_1005Metric_Pad0.72x0.64mm_HandSolder -> Resistor_SMD:R_1206_3216Metric
- R7, R8: value R -> 1.24M 1%; footprint Resistor_SMD:R_0402_1005Metric_Pad0.72x0.64mm_HandSolder -> Resistor_SMD:R_1206_3216Metric
- renumbered U3 to U1
Connections:
- net GNDPWR is gone; now on net GND: C9.2
- net GND: now also C4.2, R5.2, U1.11 (GND), U1.5 (SYNC), C1.2, C2.2, C7.2, C8.2, R9.2, U2.P$1; no longer R6.2, R8.2
- net Vhigh: now also D1.1 (K)
- net Vsupply: now also C3.1, U1.10 (VIN), U1.8 (INTVCC), C1.1, C2.1, C7.1, U2.P$7; no longer C5.1, R4.1
- net at U1.1 (VC): now also C5.1, R4.1
- net LT3757_FBX: now reaches U1.2 (FBX)
- net LT3757_FBX: now also R8.2, R9.1
- net at U1.3 (SS): now also C4.1
- net at U1.4 (RT): now also R3.1
- net at U1.6 (SENSE): now also R5.1, Q1.1 (S), Q1.2 (S), Q1.3 (S)
- net at U1.7 (GATE): now also Q1.4 (G)
- net at U1.9 (~{SHDN}/UVLO): now also R1.2, R2.1
- net at R6.1: now also Q1.5 (D), U2.P$3; no longer R7.2
- net at C6.1: now also R4.2
- net at R8.1: now also R7.2
- new net: U2.P$10, U2.P$4
- new net: D1.2 (A), U2.P$12
- new net: U2.P$5, U2.P$9
- new net: U2.P$6, U2.P$8
- new net: C8.1, R6.2
Other:
- note added: "All values still to be xreffed with datasheet"
- note added: "Two to reduce voltage drop across elements"
- note removed: "400V CAP"
- note removed: "Recommended BOM, version I would actually build first U1 LT3757AEDD#PBF or LT3757AEMSE#PBF Use the DFN if you want the smallest PCB. LT3757A is a boost/flyback/SEPIC/inverting controller, operates from 2.9 V to 40 V, drives an external low-side NMOS from its internal 7.2 V supply, and is intended for exactly this kind of topology. T1 Coilcraft DA2032-ALD This is the off-the-shelf transformer I wo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"
- company: (none) -> nacho.works
- title: (none) -> ECC83 5 to 200 V boost
- moved on the sheet: C4, C9, U1
